File: pcb/pcb-pick-plaz-aruco/pcb-pick-plaz-aruco v1.brd (EAGLE design)
At the start: 55 x 55 mm, 3 parts

Commit message: aruco & hall pcb + gerber
Parts:
- removed C1000: (no value), passives:0603_CAP
- removed R1000: (no value), passives:0603-RES
- removed U$1: LOGO-TOBENG-1MM, ftobler:TOBENG-1MM
- added V1, V2, V3, V4, V5, V6, V7, V8: FIDUCIAL2MM, ftobler:FIDUCIAL_2MM
Other:
- board text added: "pcb-pick-plaz-aruco v1 - 2021"
Changed lines of the file:
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@@
 <layer number="112" name="tSilk" color="7" fill="1" visible="no" active="yes"/>
 <layer number="113" name="ReferenceLS" color="7" fill="1" visible="no" active="no"/>
+<layer number="114" name="FRNTMAAT1" color="7" fill="1" visible="yes" active="yes"/>
+<layer number="115" name="FRNTMAAT2" color="7" fill="1" visible="yes" active="yes"/>
 <layer number="116" name="Patch_BOT" color="9" fill="4" visible="yes" active="yes"/>
+<layer number="117" name="BACKMAAT1" color="7" fill="1" visible="yes" active="yes"/>
 <layer number="118" name="Rect_Pads" color="7" fill="1" visible="no" active="no"/>
+<layer number="119" name="KAP_TEKEN" color="7" fill="1" visible="yes" active="yes"/>
+<layer number="120" name="KAP_MAAT1" color="7" fill="1" visible="yes" active="yes"/>
 <layer number="121" name="_tsilk" color="7" fill="1" visible="yes" active="yes"/>
 <layer number="122" name="_bsilk" color="7" fill="1" visible="yes" active="yes"/>
@@
 <layer number="128" name="_bValues" color="7" fill="1" visible="no" active="yes"/>
 <layer number="129" name="Mask" color="7" fill="1" visible="yes" active="yes"/>
+<layer number="130" name="SMDSTROOK" color="7" fill="1" visible="yes" active="yes"/>
 <layer number="131" name="tAdjust" color="7" fill="1" visible="no" active="yes"/>
 <layer number="132" name="bAdjust" color="7" fill="1" visible="no" active="yes"/>
+<layer number="133" name="bottom_silk" color="7" fill="1" visible="yes" active="yes"/>
+<layer number="134" name="silk_top" color="7" fill="1" visible="yes" active="yes"/>
+<layer number="135" name="silk_bottom" color="7" fill="1" visible="yes" active="yes"/>
+<layer number="136" name="silktop" color="7" fill="1" visible="yes" active="yes"/>
+<layer number="137" name="silkbottom" color="7" fill="1" visible="yes" active="yes"/>
 <layer number="144" name="Drill_legend" color="7" fill="1" visible="yes" active="yes"/>
+<layer number="145" name="DrillLegend_01-16" color="7" fill="1" visible="yes" active="yes"/>
+<layer number="146" name="DrillLegend_01-20" color="7" fill="1" visible="yes" active="yes"/>
 <layer number="150" name="Notes" color="7" fill="1" visible="no" active="yes"/>
 <layer number="151" name="HeatSink" color="7" fill="1" visible="yes" active="yes"/>
@@
 <layer number="154" name="FabDoc2" color="2" fill="1" visible="no" active="no"/>
 <layer number="155" name="FabDoc3" color="7" fill="15" visible="no" active="no"/>
+<layer number="166" name="AntennaArea" color="7" fill="1" visible="yes" active="yes"/>
+<layer number="168" name="4mmHeightArea" color="7" fill="1" visible="yes" active="yes"/>
 <layer number="199" name="Contour" color="7" fill="1" visible="yes" active="yes"/>
 <layer number="200" name="200bmp" color="1" fill="10" visible="yes" active="yes"/>
@@
 <rectangle x1="17.462503125" y1="49.4279" x2="20.462503125" y2="49.9279" layer="30" rot="R165"/>
 <rectangle x1="13.5988" y1="50.463175" x2="16.5988" y2="50.963175" layer="30" rot="R165"/>
+<text x="16.5" y="52.5" size="1.2" layer="21">pcb-pick-plaz-aruco v1 - 2021</text>
 </plain>
 <attributes>
@@
 </autorouter>
 <elements>
-<element name="C1000" library="passives" package="0603_CAP" value="" x="-4.9" y="12.3" smashed="yes">
-<attribute name="NAME" x="-4.9" y="13.062" size="0.889" layer="25" font="vector" ratio="12" align="bottom-center"/>
-</element>
-<element name="R1000" library="passives" package="0603-RES" value="" x="-4.95" y="9.35" smashed="yes">
-<attribute name="NAME" x="-4.95" y="9.731" size="0.889" layer="25" font="vector" ratio="12" align="bottom-center"/>
-<attribute name="VALUE" x="-4.95" y="7.953" size="1.016" layer="27" font="vector" ratio="12" align="bottom-center"/>
-</element>
-<element name="U$1" library="ftobler" package="TOBENG-1MM" value="LOGO-TOBENG-1MM" x="-4.85" y="3.9" smashed="yes"/>
+<element name="V1" library="ftobler" package="FIDUCIAL_2MM" value="FIDUCIAL2MM" x="6.5" y="2" smashed="yes"/>
+<element name="V2" library="ftobler" package="FIDUCIAL_2MM" value="FIDUCIAL2MM" x="48.5" y="2" smashed="yes"/>
+<element name="V3" library="ftobler" package="FIDUCIAL_2MM" value="FIDUCIAL2MM" x="6.5" y="53" smashed="yes"/>
+<element name="V4" library="ftobler" package="FIDUCIAL_2MM" value="FIDUCIAL2MM" x="48.5" y="53" smashed="yes"/>
+<element name="V5" library="ftobler" package="FIDUCIAL_2MM" value="FIDUCIAL2MM" x="6.5" y="2" smashed="yes" rot="MR0"/>
+<element name="V6" library="ftobler" package="FIDUCIAL_2MM" value="FIDUCIAL2MM" x="48.5" y="53" smashed="yes" rot="MR0"/>
+<element name="V7" library="ftobler" package="FIDUCIAL_2MM" value="FIDUCIAL2MM" x="48.5" y="2" smashed="yes" rot="MR0"/>
+<element name="V8" library="ftobler" package="FIDUCIAL_2MM" value="FIDUCIAL2MM" x="6.5" y="53" smashed="yes" rot="MR0"/>
 </elements>
 <signals>
