File: pcb/pcb-pick-plaz-aruco/pcb-pick-plaz-aruco v1.sch (EAGLE design)
At the start: 3 parts

Commit message: aruco & hall pcb + gerber
Parts:
- removed C1000: (no value), passives:CAPACITOR0603_CAP
- removed R1000: (no value), passives:RESISTOR0603_RES
- removed U$1: LOGO-TOBENG-1MM, ftobler:LOGO-TOBENG-1MM
- added V1, V2, V3, V4, V5, V6, V7, V8: FIDUCIAL2MM, ftobler:FIDUCIAL2MM
