File: pcb/pcb-pick-plaz-hall/pcb-pick-plaz-hall v1.brd (EAGLE design)
At the start: 71 x 53 mm, 13 parts, among them IC1 A1203UA, IC2 A1203LH, X1 04-JST-B4B-XH-A, X2 04-JST-B4B-XH-A

Commit message: aruco & hall pcb + gerber
Other:
- board text added: "pcb-pick-plaz-hall v1 by ftobler 2021"
Changed lines of the file:
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@@
 <text x="-0.25" y="-5.5" size="0.8" layer="29" font="vector">V2</text>
 <text x="52.5" y="43.25" size="0.8" layer="29" font="vector">V3</text>
+<text x="39.5" y="28.75" size="1.778" layer="22" rot="MR0">pcb-pick-plaz-hall v1
+by ftobler 2021</text>
 </plain>
 <attributes>
@@
 </drawing>
 <compatibility>
+<note version="6.3" minversion="6.2.2" severity="warning">
+Since Version 6.2.2 text objects can contain more than one line,
+which will not be processed correctly with this version.
+</note>
 <note version="8.2" severity="warning">
 Since Version 8.2, EAGLE supports online libraries. The ids
